Commit message: Add realsense to sim

File: catkin_ws/src/fmauch_universal_robot/ur_description/urdf/inc/ur_common.xacro (robot description, xacro)
@@ -193,4 +193,9 @@
     <xacro:property name="wrist_3_collision_mesh" value="${wrist_3_mesh['collision']['mesh']}" scope="parent"/>
     <xacro:property name="wrist_3_visual_offset" value="${wrist_3_mesh['visual_offset']}" scope="parent"/>
+    <xacro:property name="ur_d435_mesh" value="${sec_mesh_files['ur_d435']}"/>
+    <xacro:property name="ur_d435_visual_mesh" value="${ur_d435_mesh['visual']['mesh']}" scope="parent"/>
+    <xacro:property name="ur_d435_visual_material_name" value="${ur_d435_mesh['visual']['material']['name']}" scope="parent"/>
+    <xacro:property name="ur_d435_visual_material_color" value="${ur_d435_mesh['visual']['material']['color']}" scope="parent"/>
+    <xacro:property name="ur_d435_visual_offset" value="${ur_d435_mesh['visual_offset']}" scope="parent"/>
   </xacro:macro>
 </robot>

File: catkin_ws/src/fmauch_universal_robot/ur_description/urdf/inc/ur_macro.xacro (robot description, xacro)
@@ -44,5 +44,5 @@
   <xacro:include filename="$(find ur_description)/urdf/inc/ur_transmissions.xacro" />
   <xacro:include filename="$(find ur_description)/urdf/inc/ur_common.xacro" />
-  <xacro:include filename="$(find realsense2_description)/urdf/_d435.gazebo.xacro"/>
+  <xacro:include filename="$(find realsense2_description)/urdf/_d435.urdf.xacro" />
   <xacro:macro name="ur_robot" params="
     prefix
@@ -207,4 +207,18 @@
       </xacro:cylinder_inertial>
     </link>
+  <xacro:sensor_d435 name="camera_d435" topics_ns="camera_d435" parent="${prefix}wrist_3_link" publish_pointcloud="true">
+    <origin xyz="0 0 ${ur_d435_visual_offset}" rpy="${pi/2} 0 0" />
+  </xacro:sensor_d435>
+    <!-- <link name="${prefix}ur_d435_link">
+      <visual>
+        <origin xyz="0 0 ${ur_d435_visual_offset}" rpy="${pi/2} 0 0"/>
+        <geometry>
+          <mesh filename="${ur_d435_visual_mesh}"/>
+        </geometry>
+        <material name="${ur_d435_visual_material_name}">
+          <color rgba="${ur_d435_visual_material_color}"/>
+        </material>
+      </visual>
+    </link> -->
     <!-- joints: main serial chain -->
     <joint name="${prefix}base_link-base_link_inertia" type="fixed">
@@ -290,4 +304,10 @@
       <dynamics damping="0" friction="0"/>
     </joint>
+    <!-- <joint name="${prefix}ur_d435_joint" type="fixed">
+      <parent link="${prefix}wrist_3_link" />
+      <child link="${prefix}ur_d435_link" />
+      <origin xyz="0 0 0" rpy="0 0 0" />
+      <axis xyz="0 0 1" />
+    </joint> -->
     <!-- ROS-Industrial 'base' frame: base_link to UR 'Base' Coordinates transform -->
     <link name="${prefix}base"/>

File: catkin_ws/src/fmauch_universal_robot/ur_description/urdf/inc/ur_transmissions.xacro (robot description, xacro)
@@ -61,4 +61,10 @@
       </actuator>
     </transmission>
+    <transmission name="${prefix}ur_d435_trans">
+      <type>transmission_interface/SimpleTransmission</type>
+      <joint name="${prefix}ur_d435_joint">
+        <hardwareInterface>${hw_interface}</hardwareInterface>
+      </joint>
+    </transmission>
   </xacro:macro>
 </robot>

Commit message: Sensor update, benchmark

File: catkin_ws/src/fmauch_universal_robot/ur_description/urdf/inc/ur_common.xacro (robot description, xacro)
@@ -193,9 +193,9 @@
     <xacro:property name="wrist_3_collision_mesh" value="${wrist_3_mesh['collision']['mesh']}" scope="parent"/>
     <xacro:property name="wrist_3_visual_offset" value="${wrist_3_mesh['visual_offset']}" scope="parent"/>
-    <xacro:property name="ur_d435_mesh" value="${sec_mesh_files['ur_d435']}"/>
-    <xacro:property name="ur_d435_visual_mesh" value="${ur_d435_mesh['visual']['mesh']}" scope="parent"/>
-    <xacro:property name="ur_d435_visual_material_name" value="${ur_d435_mesh['visual']['material']['name']}" scope="parent"/>
-    <xacro:property name="ur_d435_visual_material_color" value="${ur_d435_mesh['visual']['material']['color']}" scope="parent"/>
-    <xacro:property name="ur_d435_visual_offset" value="${ur_d435_mesh['visual_offset']}" scope="parent"/>
+    <xacro:property name="ur_d415_mesh" value="${sec_mesh_files['ur_d415']}"/>
+    <xacro:property name="ur_d415_visual_mesh" value="${ur_d415_mesh['visual']['mesh']}" scope="parent"/>
+    <xacro:property name="ur_d415_visual_material_name" value="${ur_d415_mesh['visual']['material']['name']}" scope="parent"/>
+    <xacro:property name="ur_d415_visual_material_color" value="${ur_d415_mesh['visual']['material']['color']}" scope="parent"/>
+    <xacro:property name="ur_d415_visual_offset" value="${ur_d415_mesh['visual_offset']}" scope="parent"/>
   </xacro:macro>
 </robot>

File: catkin_ws/src/fmauch_universal_robot/ur_description/urdf/inc/ur_macro.xacro (robot description, xacro)
@@ -44,5 +44,5 @@
   <xacro:include filename="$(find ur_description)/urdf/inc/ur_transmissions.xacro" />
   <xacro:include filename="$(find ur_description)/urdf/inc/ur_common.xacro" />
-  <xacro:include filename="$(find realsense2_description)/urdf/_d435.urdf.xacro" />
+  <xacro:include filename="$(find realsense2_description)/urdf/_d415.urdf.xacro" />
   <xacro:macro name="ur_robot" params="
     prefix
@@ -207,15 +207,15 @@
       </xacro:cylinder_inertial>
     </link>
-  <xacro:sensor_d435 name="camera_d435" topics_ns="camera_d435" parent="${prefix}wrist_3_link" publish_pointcloud="true">
-    <origin xyz="0 0 ${ur_d435_visual_offset}" rpy="${pi/2} ${-pi/2} 0" />
-  </xacro:sensor_d435>
-    <!-- <link name="${prefix}ur_d435_link">
-      <visual>
-        <origin xyz="0 0 ${ur_d435_visual_offset}" rpy="${pi/2} 0 0"/>
-        <geometry>
-          <mesh filename="${ur_d435_visual_mesh}"/>
-        </geometry>
-        <material name="${ur_d435_visual_material_name}">
-          <color rgba="${ur_d435_visual_material_color}"/>
+  <xacro:sensor_d415 name="camera_d415" topics_ns="camera_d415" parent="${prefix}wrist_3_link" publish_pointcloud="true">
+    <origin xyz="0 0 ${ur_d415_visual_offset}" rpy="${pi/2} ${-pi/2} 0" />
+  </xacro:sensor_d415>
+    <!-- <link name="${prefix}ur_d415_link">
+      <visual>
+        <origin xyz="0 0 ${ur_d415_visual_offset}" rpy="${pi/2} 0 0"/>
+        <geometry>
+          <mesh filename="${ur_d415_visual_mesh}"/>
+        </geometry>
+        <material name="${ur_d415_visual_material_name}">
+          <color rgba="${ur_d415_visual_material_color}"/>
         </material>
       </visual>
@@ -304,7 +304,7 @@
       <dynamics damping="0" friction="0"/>
     </joint>
-    <!-- <joint name="${prefix}ur_d435_joint" type="fixed">
+    <!-- <joint name="${prefix}ur_d415_joint" type="fixed">
       <parent link="${prefix}wrist_3_link" />
-      <child link="${prefix}ur_d435_link" />
+      <child link="${prefix}ur_d415_link" />
       <origin xyz="0 0 0" rpy="0 0 0" />
       <axis xyz="0 0 1" />

File: catkin_ws/src/fmauch_universal_robot/ur_description/urdf/inc/ur_transmissions.xacro (robot description, xacro)
@@ -61,7 +61,7 @@
       </actuator>
     </transmission>
-    <transmission name="${prefix}ur_d435_trans">
+    <transmission name="${prefix}ur_d415_trans">
       <type>transmission_interface/SimpleTransmission</type>
-      <joint name="${prefix}ur_d435_joint">
+      <joint name="${prefix}ur_d415_joint">
         <hardwareInterface>${hw_interface}</hardwareInterface>
       </joint>

File: catkin_ws/src/realsense2_description/urdf/_d415.urdf.xacro (robot description, xacro)
@@ -7,5 +7,7 @@
 -->
 <robot name="sensor_d415" xmlns:xacro="http://ros.org/wiki/xacro">
-  <xacro:macro name="sensor_d415" params="name:=camera parent *origin">
+<!--File includes-->
+  <xacro:include filename="$(find realsense2_description)/urdf/_d415.gazebo.xacro"/>
+  <xacro:macro name="sensor_d415" params="name:=camera topics_ns:=camera parent *origin publish_pointcloud:=true">
     <xacro:property name="M_PI" value="3.1415926535897931" />
     <!-- The following values are approximate, and the camera node
@@ -115,4 +117,6 @@
     </joint>
     <link name="${name}_color_optical_frame"/>
+        <!-- Realsense Gazebo Plugin -->
+    <xacro:gazebo_d415 camera_name="${name}" reference_link="${name}_link" topics_ns="${topics_ns}" depth_optical_frame="${name}_depth_optical_frame" color_optical_frame="${name}_color_optical_frame" infrared1_optical_frame="${name}_left_ir_optical_frame" infrared2_optical_frame="${name}_right_ir_optical_frame" publish_pointcloud="${publish_pointcloud}"/>
   </xacro:macro>
 </robot>
