Commit message: Set params

File: catkin_ws/src/fmauch_universal_robot/ur_description/urdf/inc/ur_macro.xacro (robot description, xacro)
@@ -208,5 +208,5 @@
     </link>
   <xacro:sensor_d435 name="camera_d435" topics_ns="camera_d435" parent="${prefix}wrist_3_link" publish_pointcloud="true">
-    <origin xyz="0 0 ${ur_d435_visual_offset}" rpy="${pi/2} 0 0" />
+    <origin xyz="0 0 ${ur_d435_visual_offset}" rpy="${pi/2} ${-pi/2} 0" />
   </xacro:sensor_d435>
     <!-- <link name="${prefix}ur_d435_link">

File: catkin_ws/src/realsense2_description/urdf/_d435.gazebo.xacro (robot description, xacro)
@@ -41,7 +41,7 @@
           </noise>
         </camera>
-        <always_on>1</always_on>
+        <always_on>0</always_on>
         <update_rate>30</update_rate>
-        <visualize>1</visualize>
+        <visualize>0</visualize>
       </sensor>
       <sensor name="${camera_name}ired1" type="camera">
@@ -63,5 +63,5 @@
           </noise>
         </camera>
-        <always_on>1</always_on>
+        <always_on>0</always_on>
         <update_rate>90</update_rate>
         <visualize>0</visualize>
@@ -85,5 +85,5 @@
           </noise>
         </camera>
-        <always_on>1</always_on>
+        <always_on>0</always_on>
         <update_rate>90</update_rate>
         <visualize>0</visualize>

Commit message: feat: octomapping with longer cable using l515

File: catkin_ws/src/fmauch_universal_robot/ur_description/urdf/inc/ur_macro.xacro (robot description, xacro)
@@ -44,5 +44,5 @@
   <xacro:include filename="$(find ur_description)/urdf/inc/ur_transmissions.xacro" />
   <xacro:include filename="$(find ur_description)/urdf/inc/ur_common.xacro" />
-  <xacro:include filename="$(find realsense2_description)/urdf/_d435.urdf.xacro" />
+  <xacro:include filename="$(find realsense2_description)/urdf/_d415.urdf.xacro" />
   <xacro:macro name="ur_robot" params="
     prefix
@@ -206,8 +206,8 @@
         <origin xyz="0.0 0.0 ${-0.5 * wrist_3_inertia_length}" rpy="0 0 0" />
       </xacro:cylinder_inertial>
-    </link>
-  <xacro:sensor_d435 name="camera_d435" topics_ns="camera_d435" parent="${prefix}wrist_3_link" publish_pointcloud="true">
-    <origin xyz="0 0 ${ur_d435_visual_offset}" rpy="${pi/2} ${-pi/2} 0" />
-  </xacro:sensor_d435>
+      <xacro:sensor_d415 name="camera_d415" topics_ns="camera_d415" parent="${prefix}wrist_3_link" publish_pointcloud="true">
+        <origin xyz="0 0 ${ur_d415_visual_offset}" rpy="${pi/2} ${-pi/2} 0" />
+      </xacro:sensor_d415>
+    </link>
     <!-- <link name="${prefix}ur_d435_link">
       <visual>

File: catkin_ws/src/realsense2_description/urdf/_d415.urdf.xacro (robot description, xacro)
@@ -7,5 +7,5 @@
 -->
 <robot name="sensor_d415" xmlns:xacro="http://ros.org/wiki/xacro">
-  <xacro:macro name="sensor_d415" params="name:=camera parent *origin">
+  <xacro:macro name="sensor_d415" params="name:=camera topics_ns:=camera parent *origin publish_pointcloud:=true">
     <xacro:property name="M_PI" value="3.1415926535897931" />
     <!-- The following values are approximate, and the camera node
